Commit message: new updates

File: install/uav_gazebo/share/uav_gazebo/urdf/uav_sensors.urdf (robot description, URDF)
Before this commit: robot uav_sensors, 19 links, 18 joints
Links:
- removed link ground_truth/odometry_sensorgt_link
- added link odom, mass 1e-02
Joints:
- removed joint ground_truth/odometry_sensorgt_joint
- added joint odom_joint: type fixed, parent odom, child base_footprint, axis 0 0 1, limit lower=0 upper=0 effort=0 velocity=0
- joint imu_joint: type revolute -> fixed
